Commit message: renamed moveit config package

File: my_robot_cell/my_robot_cell_moveit_config/config/my_robot_cell.ros2_control.xacro (robot description, xacro)
@@ -1,5 +1,5 @@
 <?xml version="1.0"?>
 <robot xmlns:xacro="http://www.ros.org/wiki/xacro">
-    <xacro:macro name="shared_workspace_ros2_control" params="name initial_positions_file">
+    <xacro:macro name="my_robot_cell_ros2_control" params="name initial_positions_file">
         <xacro:property name="initial_positions" value="${load_yaml(initial_positions_file)['initial_positions']}"/>
         <ros2_control name="${name}" type="system">
