Commit message: changed table mesh

File: my_robot_cell/my_robot_cell_description/urdf/my_robot_cell.urdf.xacro (robot description, xacro)
@@ -20,5 +20,5 @@
     <visual>
       <geometry>
-        <mesh filename="package://my_robot_cell_description/meshes/171005_Motek_Tisch.dae"/>
+        <mesh filename="package://my_robot_cell_description/meshes/fzi_table.dae"/>
       </geometry>
       <origin rpy="0 0 0" xyz="0.75 0.5 -1"/>
@@ -27,5 +27,5 @@
     <collision>
       <geometry>
-        <mesh filename="package://my_robot_cell_description/meshes/171005_Motek_Tisch.dae"/>
+        <mesh filename="package://my_robot_cell_description/meshes/fzi_table.dae"/>
       </geometry>
       <origin rpy="0 0 0" xyz="0.75 0.5 -1"/>
@@ -89,5 +89,5 @@
     input_recipe_filename="$(arg ur_input_recipe_filename)"
   >
-    <origin xyz="0 0 0" rpy="0 0 ${pi}" />
+    <origin xyz="0 -0.05 0" rpy="0 0 ${pi}" />
   </xacro:ur_robot>
 </robot>

Commit message: Use a nicer UR background for the wall
This also adds the requirement to update licensing information of the package.

File: my_robot_cell/my_robot_cell_description/urdf/my_robot_cell.urdf.xacro (robot description, xacro)
@@ -55,5 +55,5 @@
     <visual>
       <geometry>
-        <box size="3 0.1 2.5"/>
+        <mesh filename="package://my_robot_cell_description/meshes/wall.dae"/>
       </geometry>
       <material name="white"/>
@@ -61,5 +61,5 @@
     <collision>
       <geometry>
-        <box size="3 0.1 2.5"/>
+        <box size="4.44 0.1 2.5"/>
       </geometry>
     </collision>
@@ -68,5 +68,5 @@
     <parent link="base_link"/>
     <child link="wall"/>
-    <origin xyz="0.75 1.5 0.5"/>
+    <origin xyz="1.25 1.5 0.5"/>
   </joint>
   <link name="robot_position"/>

Commit message: Update my_robot_cell/my_robot_cell_description/urdf/my_robot_cell.urdf.xacro
Co-authored-by: Felix Exner (fexner) <felix_mauch@web.de>

File: my_robot_cell/my_robot_cell_description/urdf/my_robot_cell.urdf.xacro (robot description, xacro)
@@ -24,5 +24,4 @@
       <origin rpy="0 0 0" xyz="0.75 0.5 -1"/>
     </visual>
-    <material name="black"/>
     <collision>
       <geometry>

Commit message: Update my_robot_cell/my_robot_cell_description/urdf/my_robot_cell.urdf.xacro
Co-authored-by: Felix Exner (fexner) <felix_mauch@web.de>

File: my_robot_cell/my_robot_cell_description/urdf/my_robot_cell.urdf.xacro (robot description, xacro)
@@ -56,5 +56,4 @@
         <mesh filename="package://my_robot_cell_description/meshes/wall.dae"/>
       </geometry>
-      <material name="white"/>
     </visual>
     <collision>

Commit message: renamed links

File: my_robot_cell/my_robot_cell_description/urdf/my_robot_cell.urdf.xacro (robot description, xacro)
@@ -12,10 +12,10 @@
   <xacro:arg name="ur_input_recipe_filename" default="$(find ur_robot_driver)/resources/rtde_output_recipe.txt"/>
   <link name="world"/>
-  <joint name="base_link_to_world" type="fixed">
+  <joint name="table_to_world" type="fixed">
     <parent link="world"/>
-    <child link="base_link"/>
+    <child link="table"/>
     <origin xyz="0 0 1"/>
   </joint>
-  <link name="base_link">
+  <link name="table">
     <visual>
       <geometry>
@@ -44,5 +44,5 @@
   </link>
   <joint name="base_to_monitor" type="fixed">
-    <parent link="base_link"/>
+    <parent link="table"/>
     <child link="monitor"/>
     <origin xyz="0.2 0.6 0"/>
@@ -64,12 +64,12 @@
   </link>
   <joint name="base_to_wall" type="fixed">
-    <parent link="base_link"/>
+    <parent link="table"/>
     <child link="wall"/>
     <origin xyz="1.25 1.5 0.5"/>
   </joint>
-  <link name="robot_position"/>
-  <joint name="base_to_robot_position" type="fixed">
-    <parent link="base_link"/>
-    <child link="robot_position"/>
+  <link name="robot_mount"/>
+  <joint name="base_to_robot_mount" type="fixed">
+    <parent link="table"/>
+    <child link="robot_mount"/>
     <origin xyz="0.845 0.9 0" rpy="0 0 0" />
   </joint>
@@ -77,5 +77,5 @@
     name="$(arg ur_type)"
     tf_prefix="$(arg ur_type)_"
-    parent="robot_position"
+    parent="robot_mount"
     robot_ip="$(arg robot_ip)"
     joint_limits_parameters_file="$(arg joint_limit_params)"
